File: gse_connector_board_inner/gse_connector_board.kicad_sch (KiCad schematic)
At the start: 10 parts, among them J1 arming_connector, J2 gse_com_connector, J3 chg_connector, J4 Conn_02x03_Top_Bottom, J5 Conn_02x02_Top_Bottom

Commit message: adapted footprint again
Parts:
- D1: KiLib_Generator (none) -> package/gullwing
- J2: footprint custom_parts:4_pin_mag_con_flat -> gse_inner_custom:4_pin_mag_con_flat_mv_adapt
- J3: renamed from J1; footprint custom_parts:4_pin_mag_con_flat -> gse_inner_custom:4_pin_mag_con_flat_mv_adapt
- J5: renamed from J3; footprint custom_parts:4_pin_mag_con_flat -> gse_inner_custom:4_pin_mag_con_flat_mv_adapt
- R1: renamed from R24; KiLib_Generator (none) -> SMD_2terminal_chip_molded
- renumbered JP1 to 120Ω1, J5 to J1
Changed lines of the file:
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@@
 		(in_pos_files yes)
 		(dnp no)
-		(property "Reference" "R24"
+		(property "Reference" "R1"
 			(at 63.246 45.466 0)
 			(show_name no)
@@
 			)
 		)
+		(property "KiLib_Generator" "SMD_2terminal_chip_molded"
+			(at 64.77 44.45 0)
+			(hide yes)
+			(show_name no)
+			(do_not_autoplace no)
+			(effects
+				(font
+					(size 1.27 1.27)
+				)
+			)
+		)
 		(pin "1"
 		)
@@
 			(project "gse_connector_board"
 				(path "/df677c4e-51be-471c-a547-b22db5b9f5a1"
-					(reference "R24")
+					(reference "R1")
 					(unit 1)
 				)
@@
 		(dnp no)
 		(fields_autoplaced yes)
-		(property "Reference" "#PWR067"
+		(property "Reference" "#PWR06"
 			(at 41.91 58.42 0)
 			(hide yes)
@@
 			(project "gse_connector_board"
 				(path "/df677c4e-51be-471c-a547-b22db5b9f5a1"
-					(reference "#PWR067")
+					(reference "#PWR06")
 					(unit 1)
 				)
@@
 			)
 		)
+		(property "KiLib_Generator" "package/gullwing"
+			(at 41.91 46.99 0)
+			(hide yes)
+			(show_name no)
+			(do_not_autoplace no)
+			(effects
+				(font
+					(size 1.27 1.27)
+				)
+			)
+		)
 		(pin "1"
 		)
@@
 		(dnp no)
 		(fields_autoplaced yes)
-		(property "Reference" "#PWR03"
+		(property "Reference" "#PWR08"
 			(at 54.61 87.63 0)
 			(hide yes)
@@
 			(project "gse_connector_board"
 				(path "/df677c4e-51be-471c-a547-b22db5b9f5a1"
-					(reference "#PWR03")
+					(reference "#PWR08")
 					(unit 1)
 				)
@@
 		(in_pos_files yes)
 		(dnp yes)
-		(property "Reference" "J3"
+		(property "Reference" "J5"
 			(at 90.678 77.724 0)
 			(show_name no)
@@
 			)
 		)
-		(property "Footprint" "custom_parts:4_pin_mag_con_flat"
+		(property "Footprint" "gse_inner_custom:4_pin_mag_con_flat_mv_adapt"
 			(at 92.71 82.55 0)
 			(hide yes)
@@
 			(project "gse_connector_board"
 				(path "/df677c4e-51be-471c-a547-b22db5b9f5a1"
-					(reference "J3")
+					(reference "J5")
 					(unit 1)
 				)
@@
 		(in_pos_files yes)
 		(dnp no)
-		(property "Reference" "#PWR059"
+		(property "Reference" "#PWR04"
 			(at 31.75 93.98 0)
 			(hide yes)
@@
 			(project "gse_connector_board"
 				(path "/df677c4e-51be-471c-a547-b22db5b9f5a1"
-					(reference "#PWR059")
+					(reference "#PWR04")
 					(unit 1)
 				)
@@
 		(in_pos_files yes)
 		(dnp yes)
-		(property "Reference" "J1"
+		(property "Reference" "J3"
 			(at 67.31 82.5499 0)
 			(show_name no)
@@
 			)
 		)
-		(property "Footprint" "custom_parts:4_pin_mag_con_flat"
+		(property "Footprint" "gse_inner_custom:4_pin_mag_con_flat_mv_adapt"
 			(at 66.04 82.55 0)
 			(hide yes)
@@
 			(project "gse_connector_board"
 				(path "/df677c4e-51be-471c-a547-b22db5b9f5a1"
-					(reference "J1")
+					(reference "J3")
 					(unit 1)
 				)
@@
 		(dnp no)
 		(fields_autoplaced yes)
-		(property "Reference" "#PWR051"
+		(property "Reference" "#PWR02"
 			(at 26.67 138.43 0)
 			(hide yes)
@@
 			(project "gse_connector_board"
 				(path "/df677c4e-51be-471c-a547-b22db5b9f5a1"
-					(reference "#PWR051")
+					(reference "#PWR02")
 					(unit 1)
 				)
@@
 		(in_pos_files yes)
 		(dnp no)
-		(property "Reference" "#PWR055"
+		(property "Reference" "#PWR03"
 			(at 31.75 83.82 0)
 			(hide yes)
@@
 			(project "gse_connector_board"
 				(path "/df677c4e-51be-471c-a547-b22db5b9f5a1"
-					(reference "#PWR055")
+					(reference "#PWR03")
 					(unit 1)
 				)
@@
 		(dnp no)
 		(fields_autoplaced yes)
-		(property "Reference" "J5"
+		(property "Reference" "J1"
 			(at 33.02 99.06 0)
 			(show_name no)
@@
 			(project "gse_connector_board"
 				(path "/df677c4e-51be-471c-a547-b22db5b9f5a1"
-					(reference "J5")
+					(reference "J1")
 					(unit 1)
 				)
@@
 		(dnp no)
 		(fields_autoplaced yes)
-		(property "Reference" "#PWR060"
+		(property "Reference" "#PWR05"
 			(at 35.56 105.41 0)
 			(hide yes)
@@
 			(project "gse_connector_board"
 				(path "/df677c4e-51be-471c-a547-b22db5b9f5a1"
-					(reference "#PWR060")
+					(reference "#PWR05")
 					(unit 1)
 				)
@@
 		(dnp no)
 		(fields_autoplaced yes)
-		(property "Reference" "#PWR066"
+		(property "Reference" "#PWR09"
 			(at 58.42 104.14 0)
 			(hide yes)
@@
 			(project "gse_connector_board"
 				(path "/df677c4e-51be-471c-a547-b22db5b9f5a1"
-					(reference "#PWR066")
+					(reference "#PWR09")
 					(unit 1)
 				)
@@
 		(dnp no)
 		(fields_autoplaced yes)
-		(property "Reference" "#PWR02"
+		(property "Reference" "#PWR010"
 			(at 81.28 80.01 0)
 			(hide yes)
@@
 			(project "gse_connector_board"
 				(path "/df677c4e-51be-471c-a547-b22db5b9f5a1"
-					(reference "#PWR02")
+					(reference "#PWR010")
 					(unit 1)
 				)
@@
 		(dnp no)
 		(fields_autoplaced yes)
-		(property "Reference" "#PWR01"
+		(property "Reference" "#PWR011"
 			(at 81.28 87.63 0)
 			(hide yes)
@@
 			(project "gse_connector_board"
 				(path "/df677c4e-51be-471c-a547-b22db5b9f5a1"
-					(reference "#PWR01")
+					(reference "#PWR011")
 					(unit 1)
 				)
@@
 		(dnp no)
 		(fields_autoplaced yes)
-		(property "Reference" "#PWR053"
+		(property "Reference" "#PWR07"
 			(at 64.77 80.01 0)
 			(hide yes)
@@
 			(project "gse_connector_board"
 				(path "/df677c4e-51be-471c-a547-b22db5b9f5a1"
-					(reference "#PWR053")
+					(reference "#PWR07")
 					(unit 1)
 				)
@@
 		(dnp no)
 		(fields_autoplaced yes)
-		(property "Reference" "#PWR04"
+		(property "Reference" "#PWR01"
 			(at 20.32 105.41 0)
 			(hide yes)
@@
 			(project "gse_connector_board"
 				(path "/df677c4e-51be-471c-a547-b22db5b9f5a1"
-					(reference "#PWR04")
+					(reference "#PWR01")
 					(unit 1)
 				)
@@
 			)
 		)
-		(property "Footprint" "custom_parts:4_pin_mag_con_flat"
+		(property "Footprint" "gse_inner_custom:4_pin_mag_con_flat_mv_adapt"
 			(at 36.83 82.55 0)
 			(hide yes)
@@
 		(in_pos_files yes)
 		(dnp no)
-		(property "Reference" "JP1"
+		(property "Reference" "120Ω1"
 			(at 69.85 54.356 0)
 			(show_name no)
@@
 			(project "gse_connector_board"
 				(path "/df677c4e-51be-471c-a547-b22db5b9f5a1"
-					(reference "JP1")
-					(unit 1)
-				)
+					(reference "120Ω1")
+					(unit 1)
+				)
