File: gse_connector_board_inner/gse_connector_board.kicad_sch (KiCad schematic)
At the start: 10 parts, among them J1 Conn_02x02_Top_Bottom, J2 gse_com_connector, J3 arming_connector, J4 Conn_02x03_Top_Bottom, J5 chg_connector

Commit message: final order version
Parts:
- J1, J4: now not fitted
- J2, J3, J5: footprint gse_inner_custom:4_pin_mag_con_flat_mv_adapt -> gse_inner_custom:4_pin_mag_con_mv_adapt
Changed lines of the file:
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@@
 			)
 		)
-		(property "Footprint" "gse_inner_custom:4_pin_mag_con_flat_mv_adapt"
+		(property "Footprint" "gse_inner_custom:4_pin_mag_con_mv_adapt"
 			(at 92.71 82.55 0)
 			(hide yes)
@@
 			)
 		)
-		(property "Footprint" "gse_inner_custom:4_pin_mag_con_flat_mv_adapt"
+		(property "Footprint" "gse_inner_custom:4_pin_mag_con_mv_adapt"
 			(at 66.04 82.55 0)
 			(hide yes)
@@
 		(on_board yes)
 		(in_pos_files yes)
-		(dnp no)
+		(dnp yes)
 		(fields_autoplaced yes)
 		(property "Reference" "J1"
@@
 		(on_board yes)
 		(in_pos_files yes)
-		(dnp no)
+		(dnp yes)
 		(fields_autoplaced yes)
 		(property "Reference" "J4"
@@
 			)
 		)
-		(property "Footprint" "gse_inner_custom:4_pin_mag_con_flat_mv_adapt"
+		(property "Footprint" "gse_inner_custom:4_pin_mag_con_mv_adapt"
 			(at 36.83 82.55 0)
 			(hide yes)
