File: gse_connector_board_inner/gse_connector_board.kicad_pcb (KiCad board)
At the start: 2 copper layers, 52 x 27 mm, 11 parts, among them J1 Conn_02x02_Top_Bottom, J2 gse_com_connector, J3 arming_connector, J4 Conn_02x03_Top_Bottom, J5 chg_connector

Commit message: final order version
Parts:
- J2, J3, J5: footprint gse_inner_custom:4_pin_mag_con_flat_mv_adapt -> gse_inner_custom:4_pin_mag_con_mv_adapt
- moved 120Ω1 1.68 mm to (127.2, 84.8), turned to -135 degrees
- moved J1 1.14 mm to (137.0, 82.1)
- moved R1 1.12 mm to (122.0, 85.8), turned to 135 degrees
Routing:
- net CAN_1+: track 24.2 -> 29.7 mm
- net Net-(120Ω1-A): track 3.73 -> 8.11 mm, vias 0 -> 2
- net disarm: track 8.63 -> 9.78 mm
- net arm: track 12.3 -> 13.4 mm
- net CAN_1-: track 26.5 -> 27.5 mm
- net voltage_Arm: track 22.1 -> 22.7 mm
