File: gse_connector_board_inner/gse_connector_board.kicad_pcb (KiCad board)
At the start: 2 copper layers, 52 x 27 mm, 11 parts, among them J1 arming_connector, J2 gse_com_connector, J3 chg_connector, J4 Conn_02x03_Top_Bottom, J5 Conn_02x02_Top_Bottom

Commit message: adapted footprint again
Parts:
- J2: footprint custom_parts:4_pin_mag_con_flat -> gse_inner_custom:4_pin_mag_con_flat_mv_adapt
- J3: renamed from J1; footprint custom_parts:4_pin_mag_con_flat -> gse_inner_custom:4_pin_mag_con_flat_mv_adapt
- J5: renamed from J3; footprint custom_parts:4_pin_mag_con_flat -> gse_inner_custom:4_pin_mag_con_flat_mv_adapt
- renumbered 120Ω to 120Ω1, J5 to J1, R24 to R1
Routing:
- net GND: track 15.9 -> 1.98 mm, vias 0 -> 2
Other:
- board text removed: "120Ω"
Changed lines of the file:
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@@
 		(descr "Resistor SMD 0402 (1005 Metric), square (rectangular) end terminal, IPC-7351 nominal, (Body size source: IPC-SM-782 page 72, https://www.pcb-3d.com/wordpress/wp-content/uploads/ipc-sm-782a_amendment_1_and_2.pdf)")
 		(tags "resistor")
-		(property "Reference" "R24"
+		(property "Reference" "R1"
 			(at -0.353553 -1.414214 45)
 			(layer "F.SilkS")
@@
 			(layers "F.Cu" "F.Mask" "F.Paste")
 			(roundrect_rratio 0.25)
-			(net "Net-(JP1-A)")
+			(net "Net-(120Ω1-A)")
 			(pintype "passive")
 		)
@@
 		(descr "SMD Solder Jumper, 1x1.5mm, rounded Pads, 0.3mm gap, bridged with 1 copper strip")
 		(tags "net tie solder jumper bridged")
-		(property "Reference" "120Ω"
+		(property "Reference" "120Ω1"
 			(at 3.889087 0 45)
 			(layer "F.SilkS")
@@
 			(size 1 0.5)
 			(layers "F.Cu" "F.Mask")
-			(net "Net-(JP1-A)")
+			(net "Net-(120Ω1-A)")
 			(pinfunction "A_1")
 			(pintype "passive")
@@
 		(descr "Molex Micro-Fit 3.0 Connector System, 43045-0400 (alternative finishes: 43045-040x), 2 Pins per row (https://www.molex.com/pdm_docs/sd/430450201_sd.pdf)")
 		(tags "connector Molex Micro-Fit_3.0 horizontal")
-		(property "Reference" "J5"
+		(property "Reference" "J1"
 			(at 1.5 -10.12 0)
 			(layer "F.SilkS")
@@
 		(embedded_fonts no)
 	)
-	(footprint "custom_parts:4_pin_mag_con_flat"
+	(footprint "gse_inner_custom:4_pin_mag_con_flat_mv_adapt"
 		(layer "B.Cu")
 		(at 143.000001 95.999999 180)
-		(property "Reference" "J1"
-			(at -0.249999 -0.825001 0)
+		(property "Reference" "J3"
+			(at 0 6.832654 0)
 			(unlocked yes)
 			(layer "B.SilkS")
+			(hide yes)
 			(effects
 				(font
@@
 		(duplicate_pad_numbers_are_jumpers no)
 		(fp_circle
-			(center 0.000001 2.999999)
-			(end 6.750001 2.999999)
-			(stroke
-				(width 0.1)
-				(type default)
-			)
-			(fill no)
-			(layer "B.SilkS")
-		)
-		(fp_circle
 			(center 0 3)
 			(end 6.75 3)
@@
 		)
 		(fp_text user "${REFERENCE}"
-			(at 0.000001 -2.500001 0)
+			(at 0 -2.5 0)
 			(unlocked yes)
 			(layer "B.Fab")
@@
 		)
 		(pad "1" thru_hole oval
-			(at -3.499999 2.999999 180)
+			(at -3.5 3 180)
 			(size 1.2 4.54)
 			(drill 1)
@@
 		)
 		(pad "2" thru_hole oval
-			(at -1.499999 2.999999 180)
+			(at -1.5 3 180)
 			(size 1.2 4.54)
 			(drill 1)
@@
 		)
 		(pad "3" thru_hole oval
-			(at 0.000001 2.999999 180)
+			(at 0 3 180)
 			(size 1.2 4.54)
 			(drill 1)
@@
 		)
 		(pad "4" thru_hole oval
-			(at 2.500001 2.999999 180)
+			(at 2.5 3 180)
 			(size 1.2 4.54)
 			(drill 1)
@@
 		(embedded_fonts no)
 	)
-	(footprint "custom_parts:4_pin_mag_con_flat"
+	(footprint "gse_inner_custom:4_pin_mag_con_flat_mv_adapt"
 		(layer "B.Cu")
 		(at 113 96 180)
-		(property "Reference" "J3"
-			(at 0 -0.5 0)
+		(property "Reference" "J5"
+			(at 0 6.832654 0)
 			(unlocked yes)
 			(layer "B.SilkS")
+			(hide yes)
 			(effects
 				(font
@@
 			(end 6.75 3)
 			(stroke
-				(width 0.1)
-				(type default)
+				(width 0.05)
+				(type solid)
 			)
 			(fill no)
@@
 			)
 		)
+		(fp_text user "${REFERENCE}"
+			(at 0 -2.5 0)
+			(unlocked yes)
+			(layer "B.Fab")
+			(effects
+				(font
+					(size 1 1)
+					(thickness 0.15)
+				)
+				(justify mirror)
+			)
+		)
 		(pad "1" thru_hole oval
 			(at -3.5 3 180)
@@
 		(embedded_fonts no)
 	)
-	(footprint "custom_parts:4_pin_mag_con_flat"
+	(footprint "gse_inner_custom:4_pin_mag_con_flat_mv_adapt"
 		(layer "B.Cu")
 		(at 128 90)
@@
 			(unlocked yes)
 			(layer "B.SilkS")
+			(hide yes)
 			(effects
 				(font
@@
 		)
 	)
-	(gr_text "120Ω"
-		(at 117.775 81.975 270)
-		(layer "B.SilkS")
-		(effects
-			(font
-				(size 1 1)
-				(thickness 0.15)
-			)
-			(justify left bottom mirror)
-		)
-	)
 	(gr_text "rev2"
 		(at 130.094044 74.667346 0)
@@
 	)
 	(segment
+		(start 123.360624 84.889376)
+		(end 124.389376 84.889376)
+		(width 0.2)
+		(layer "F.Cu")
+		(net "Net-(120Ω1-A)")
+	)
+	(segment
+		(start 126.040381 86.511629)
+		(end 126.040381 86.709619)
+		(width 0.2)
+		(layer "F.Cu")
+		(net "Net-(120Ω1-A)")
+	)
+	(segment
+		(start 124.389376 84.889376)
+		(end 126.040381 86.540381)
+		(width 0.2)
+		(layer "F.Cu")
+		(net "Net-(120Ω1-A)")
+	)
+	(segment
+		(start 126.040381 86.540381)
+		(end 126.040381 86.709619)
+		(width 0.2)
+		(layer "F.Cu")
+		(net "Net-(120Ω1-A)")
+	)
+	(segment
+		(start 126.5 92.057208)
+		(end 126.5 93)
+		(width 0.2)
+		(layer "F.Cu")
+		(net "CAN_1+")
+	)
+	(segment
+		(start 120.7375 83.95)
+		(end 120.95 83.95)
+		(width 0.2)
+		(layer "F.Cu")
+		(net "CAN_1+")
+	)
+	(segment
+		(start 118.597654 85.102346)
+		(end 119.75 83.95)
+		(width 0.2)
+		(layer "F.Cu")
+		(net "CAN_1+")
+	)
+	(segment
+		(start 119.75 83.95)
+		(end 120.7375 83.95)
+		(width 0.2)
+		(layer "F.Cu")
+		(net "CAN_1+")
+	)
+	(segment
+		(start 126.74 89.74)
+		(end 126.74 92.76)
+		(width 0.2)
+		(layer "F.Cu")
+		(net "CAN_1+")
+	)
+	(segment
+		(start 109.744044 85.102346)
+		(end 118.597654 85.102346)
+		(width 0.2)
+		(layer "F.Cu")
+		(net "CAN_1+")
+	)
+	(segment
+		(start 126.74 92.76)
+		(end 126.5 93)
+		(width 0.2)
+		(layer "F.Cu")
+		(net "CAN_1+")
+	)
+	(segment
+		(start 120.95 83.95)
+		(end 126.74 89.74)
+		(width 0.2)
+		(layer "F.Cu")
+		(net "CAN_1+")
+	)
+	(segment
+		(start 118.8625 83.6625)
+		(end 118.9 83.7)
+		(width 0.2)
+		(layer "F.Cu")
+		(net "GND")
+	)
+	(segment
+		(start 118.8625 83)
+		(end 117.6 83)
+		(width 0.2)
+		(layer "F.Cu")
+		(net "GND")
+	)
+	(segment
+		(start 118.8625 83)
+		(end 118.8625 83.6625)
+		(width 0.2)
+		(layer "F.Cu")
+		(net "GND")
+	)
+	(via
+		(at 117.6 83)
+		(size 0.6)
+		(drill 0.3)
+		(layers "F.Cu" "B.Cu")
+		(net "GND")
+	)
+	(via
+		(at 118.9 83.7)
+		(size 0.6)
+		(drill 0.3)
+		(layers "F.Cu" "B.Cu")
+		(net "GND")
+	)
+	(segment
 		(start 120.685154 82.102346)
 		(end 120.7375 82.05)
@@
 	)
 	(segment
-		(start 106.744044 82.102346)
-		(end 108.141698 83.5)
-		(width 0.5)
-		(layer "F.Cu")
-		(net "GND")
-	)
-	(segment
-		(start 108.141698 83.5)
-		(end 118.3625 83.5)
-		(width 0.5)
-		(layer "F.Cu")
-		(net "GND")
-	)
-	(segment
-		(start 103.744044 82.102346)
-		(end 106.744044 82.102346)
-		(width 0.5)
-		(layer "F.Cu")
-		(net "GND")
-	)
-	(segment
-		(start 118.3625 83.5)
-		(end 118.8625 83)
-		(width 0.5)
-		(layer "F.Cu")
-		(net "GND")
-	)
-	(segment
 		(start 103.844044 85.137346)
 		(end 107.374044 88.667346)
@@
 	)
 	(segment
-		(start 126.5 92.057208)
-		(end 126.5 93)
-		(width 0.2)
-		(layer "F.Cu")
-		(net "CAN_1+")
-	)
-	(segment
-		(start 120.7375 83.95)
-		(end 120.95 83.95)
-		(width 0.2)
-		(layer "F.Cu")
-		(net "CAN_1+")
-	)
-	(segment
-		(start 126.74 89.74)
-		(end 126.74 92.76)
-		(width 0.2)
-		(layer "F.Cu")
-		(net "CAN_1+")
-	)
-	(segment
-		(start 119.585154 85.102346)
-		(end 120.7375 83.95)
-		(width 0.2)
-		(layer "F.Cu")
-		(net "CAN_1+")
-	)
-	(segment
-		(start 126.74 92.76)
-		(end 126.5 93)
-		(width 0.2)
-		(layer "F.Cu")
-		(net "CAN_1+")
-	)
-	(segment
-		(start 120.95 83.95)
-		(end 126.74 89.74)
-		(width 0.2)
-		(layer "F.Cu")
-		(net "CAN_1+")
-	)
-	(segment
-		(start 109.744044 85.102346)
-		(end 119.585154 85.102346)
-		(width 0.2)
-		(layer "F.Cu")
-		(net "CAN_1+")
-	)
-	(segment
 		(start 139.6 86.6)
 		(end 139.6 83.593302)
@@
 		(net "disarm")
 	)
-	(segment
-		(start 123.360624 84.889376)
-		(end 124.389376 84.889376)
-		(width 0.2)
-		(layer "F.Cu")
-		(net "Net-(JP1-A)")
-	)
-	(segment
-		(start 126.040381 86.511629)
-		(end 126.040381 86.709619)
-		(width 0.2)
-		(layer "F.Cu")
-		(net "Net-(JP1-A)")
-	)
-	(segment
-		(start 124.389376 84.889376)
-		(end 126.040381 86.540381)
-		(width 0.2)
-		(layer "F.Cu")
-		(net "Net-(JP1-A)")
-	)
-	(segment
-		(start 126.040381 86.540381)
-		(end 126.040381 86.709619)
-		(width 0.2)
-		(layer "F.Cu")
-		(net "Net-(JP1-A)")
-	)
 	(zone

Commit message: final touches
Parts:
- removed 120Ω1: SolderJumper_2_Bridged, Jumper:SolderJumper-2_P1.3mm_Bridged_RoundedPad1.0x1.5mm
- added 120Ω: SolderJumper_2_Bridged, Jumper:SolderJumper-2_P1.3mm_Bridged_RoundedPad1.0x1.5mm, B.Cu at (124.5, 84.0)
- added R2: 2.2k, Resistor_SMD:R_0603_1608Metric_Pad0.98x0.95mm_HandSolder, F.Cu at (132.9, 85.5)
- added U1: CPC1114N, Package_SO:SOP-4_3.8x4.1mm_P2.54mm, F.Cu at (128.3, 81.2)
- R1: footprint Resistor_SMD:R_0402_1005Metric -> Resistor_SMD:R_0603_1608Metric_Pad0.98x0.95mm_HandSolder
- moved D1 9.78 mm to (128.7, 87.0), turned to 0 degrees
- moved J4 3.50 mm to (107.2, 82.1)
- moved G*** 3.35 mm to (118.7, 77.2)
- moved R1 1.58 mm to (121.5, 84.8), turned to 90 degrees
- moved J1 0.50 mm to (137.6, 82.1)
Routing:
- net +V_EXT: track 0.00 -> 20.9 mm
- net CAN_1+: track 24.2 -> 28.4 mm
- net CHG: track 20.1 -> 16.7 mm
- net Net-(120Ω1-B): track 0.00 -> 3.20 mm, vias 0 -> 1
- net Net-(R2-Pad2): track 0.00 -> 2.75 mm
- net CAN_1-: track 26.5 -> 29.0 mm
- net GND: track 1.98 -> 0.00 mm, vias 2 -> 0
- net Net-(120Ω1-A): track 3.73 -> 3.43 mm, vias 0 -> 1
- net GND_Arm: vias 0 -> 7
- added copper zone on F.Cu, net GND
- added copper zone on F.Cu, net GND_Arm
Other:
- board text added: "GSE Connector board"
- board text added: "rev2.1"
- board text removed: "GSE Connectorboard"
- board text removed: "rev2"

Commit message: final ordered version
Parts:
- J2, J3, J5: footprint gse_inner_custom:4_pin_mag_con_flat_mv_adapt -> gse_inner_custom:4_pin_mag_con_mv_adapt
- renumbered 120Ω to 120Ω1
Routing:
- net CAN_1+: track 28.4 -> 29.4 mm
- net CAN_1-: track 29.0 -> 29.5 mm
