File: gse_connector_board_outer/gse_connector_board_outer.kicad_pcb (KiCad board)
At the start: 2 copper layers, 59 x 27 mm, 11 parts, among them J1 arming_connector, J2 gse_com_connector, J3 chg_connector, J4 Conn_02x04_Top_Bottom, J5 Conn_02x02_Top_Bottom, J7 Conn_02x02_Top_Bottom, J8 Conn_02x02_Top_Bottom

Commit message: final order version
Parts:
- J1, J2, J3: footprint custom_parts:4_pin_mag_con_mv_adapt -> custom_parts:4_pin_mag_con_flat_mv_adapt
- moved G*** 2.30 mm to (148.5, 90.5)
Changed lines of the file:
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@@
 	(footprint "frodo_io_module:rapid_logo"
 		(layer "F.Cu")
-		(at 146.25 91)
+		(at 148.5 90.5)
 		(property "Reference" "G***"
 			(at 0 0 0)
@@
 		(embedded_fonts no)
 	)
-	(footprint "custom_parts:4_pin_mag_con_mv_adapt"
+	(footprint "custom_parts:4_pin_mag_con_flat_mv_adapt"
 		(layer "F.Cu")
 		(at 133 111)
 		(property "Reference" "J2"
-			(at -0.3 -6.2 0)
+			(at 0 -6.832654 0)
 			(unlocked yes)
 			(layer "F.SilkS")
@@
 		)
 		(property "Value" "gse_com_connector"
-			(at 0.15 1 180)
+			(at 0 1 0)
 			(unlocked yes)
 			(layer "F.Fab")
@@
 		)
 		(property "Datasheet" ""
-			(at 0 0 180)
+			(at 0 0 0)
 			(unlocked yes)
 			(layer "F.Fab")
@@
 		)
 		(property "Description" "Generic connector, single row, 01x04, script generated"
-			(at 0 0 180)
+			(at 0 0 0)
 			(unlocked yes)
 			(layer "F.Fab")
@@
 			(layer "F.SilkS")
 		)
+		(fp_text user "${REFERENCE}"
+			(at 0 2.5 0)
+			(unlocked yes)
+			(layer "F.Fab")
+			(effects
+				(font
+					(size 1 1)
+					(thickness 0.15)
+				)
+			)
+		)
+		(fp_text user "${REFERENCE}"
+			(at 0 2.5 0)
+			(unlocked yes)
+			(layer "F.Fab")
+			(effects
+				(font
+					(size 1 1)
+					(thickness 0.15)
+				)
+			)
+		)
 		(pad "1" thru_hole oval
-			(at -3.7 -3 180)
+			(at -3.5 -3)
 			(size 1.2 4.54)
-			(drill oval 0.8 1.75)
+			(drill 1)
 			(layers "*.Cu" "*.Mask")
 			(remove_unused_layers no)
@@
 		)
 		(pad "2" thru_hole oval
-			(at -1.5 -3 180)
+			(at -1.5 -3)
 			(size 1.2 4.54)
-			(drill oval 0.8 1.75)
+			(drill 1)
 			(layers "*.Cu" "*.Mask")
 			(remove_unused_layers no)
@@
 		)
 		(pad "3" thru_hole oval
-			(at 0 -3 180)
-			(size 1.4 4.54)
+			(at 0 -3)
+			(size 1.2 4.54)
 			(drill 1)
 			(layers "*.Cu" "*.Mask")
@@
 		)
 		(pad "4" thru_hole oval
-			(at 2.5 -3 180)
+			(at 2.5 -3)
 			(size 1.2 4.54)
-			(drill oval 0.8 1.75)
+			(drill 1)
 			(layers "*.Cu" "*.Mask")
 			(remove_unused_layers no)
@@
 		(embedded_fonts no)
 	)
-	(footprint "custom_parts:4_pin_mag_con_mv_adapt"
+	(footprint "custom_parts:4_pin_mag_con_flat_mv_adapt"
 		(layer "F.Cu")
 		(at 148 111)
 		(property "Reference" "J1"
-			(at -0.3 -6.2 0)
+			(at 0 -6.832654 0)
 			(unlocked yes)
 			(layer "F.SilkS")
@@
 		)
 		(property "Value" "arming_connector"
-			(at 0.15 1 180)
+			(at 0 1 0)
 			(unlocked yes)
 			(layer "F.Fab")
@@
 		)
 		(property "Datasheet" ""
-			(at 0 0 180)
+			(at 0 0 0)
 			(unlocked yes)
 			(layer "F.Fab")
@@
 		)
 		(property "Description" "Generic connector, single row, 01x04, script generated"
-			(at 0 0 180)
+			(at 0 0 0)
 			(unlocked yes)
 			(layer "F.Fab")
@@
 			(layer "F.SilkS")
 		)
+		(fp_text user "${REFERENCE}"
+			(at 0 2.5 0)
+			(unlocked yes)
+			(layer "F.Fab")
+			(effects
+				(font
+					(size 1 1)
+					(thickness 0.15)
+				)
+			)
+		)
+		(fp_text user "${REFERENCE}"
+			(at 0 2.5 0)
+			(unlocked yes)
+			(layer "F.Fab")
+			(effects
+				(font
+					(size 1 1)
+					(thickness 0.15)
+				)
+			)
+		)
 		(pad "1" thru_hole oval
-			(at -3.7 -3 180)
+			(at -3.5 -3)
 			(size 1.2 4.54)
-			(drill oval 0.8 1.75)
+			(drill 1)
 			(layers "*.Cu" "*.Mask")
 			(remove_unused_layers no)
@@
 		)
 		(pad "2" thru_hole oval
-			(at -1.5 -3 180)
+			(at -1.5 -3)
 			(size 1.2 4.54)
-			(drill oval 0.8 1.75)
+			(drill 1)
 			(layers "*.Cu" "*.Mask")
 			(remove_unused_layers no)
@@
 		)
 		(pad "3" thru_hole oval
-			(at 0 -3 180)
-			(size 1.4 4.54)
+			(at 0 -3)
+			(size 1.2 4.54)
 			(drill 1)
 			(layers "*.Cu" "*.Mask")
@@
 		)
 		(pad "4" thru_hole oval
-			(at 2.5 -3 180)
+			(at 2.5 -3)
 			(size 1.2 4.54)
-			(drill oval 0.8 1.75)
+			(drill 1)
 			(layers "*.Cu" "*.Mask")
 			(remove_unused_layers no)
@@
 		(embedded_fonts no)
 	)
-	(footprint "custom_parts:4_pin_mag_con_mv_adapt"
+	(footprint "custom_parts:4_pin_mag_con_flat_mv_adapt"
 		(layer "F.Cu")
 		(at 118 111)
 		(property "Reference" "J3"
-			(at -0.3 -6.2 0)
+			(at 0 -6.832654 0)
 			(unlocked yes)
 			(layer "F.SilkS")
@@
 		)
 		(property "Value" "chg_connector"
-			(at 0.15 1 180)
+			(at 0 1 0)
 			(unlocked yes)
 			(layer "F.Fab")
@@
 		)
 		(property "Datasheet" ""
-			(at 0 0 180)
+			(at 0 0 0)
 			(unlocked yes)
 			(layer "F.Fab")
@@
 		)
 		(property "Description" "Generic connector, single row, 01x04, script generated"
-			(at 0 0 180)
+			(at 0 0 0)
 			(unlocked yes)
 			(layer "F.Fab")
@@
 			(layer "F.SilkS")
 		)
+		(fp_text user "${REFERENCE}"
+			(at 0 2.5 0)
+			(unlocked yes)
+			(layer "F.Fab")
+			(effects
+				(font
+					(size 1 1)
+					(thickness 0.15)
+				)
+			)
+		)
+		(fp_text user "${REFERENCE}"
+			(at 0 2.5 0)
+			(unlocked yes)
+			(layer "F.Fab")
+			(effects
+				(font
+					(size 1 1)
+					(thickness 0.15)
+				)
+			)
+		)
 		(pad "1" thru_hole oval
-			(at -3.7 -3 180)
+			(at -3.5 -3)
 			(size 1.2 4.54)
-			(drill oval 0.8 1.75)
+			(drill 1)
 			(layers "*.Cu" "*.Mask")
 			(remove_unused_layers no)
@@
 		)
 		(pad "2" thru_hole oval
-			(at -1.5 -3 180)
+			(at -1.5 -3)
 			(size 1.2 4.54)
-			(drill oval 0.8 1.75)
+			(drill 1)
 			(layers "*.Cu" "*.Mask")
 			(remove_unused_layers no)
@@
 		)
 		(pad "3" thru_hole oval
-			(at 0 -3 180)
-			(size 1.4 4.54)
+			(at 0 -3)
+			(size 1.2 4.54)
 			(drill 1)
 			(layers "*.Cu" "*.Mask")
@@
 		)
 		(pad "4" thru_hole oval
-			(at 2.5 -3 180)
+			(at 2.5 -3)
 			(size 1.2 4.54)
-			(drill oval 0.8 1.75)
+			(drill 1)
 			(layers "*.Cu" "*.Mask")
 			(remove_unused_layers no)
@@
 	)
 	(segment
-		(start 131.18098 105.98098)
-		(end 131.75 106.55)
+		(start 125.7 100.5)
+		(end 127.622718 102.422718)
 		(width 0.2)
 		(layer "F.Cu")
@@
 	)
 	(segment
-		(start 125.7 100.5)
-		(end 127.622718 102.422718)
+		(start 131.18098 105.98098)
+		(end 131.5 106.3)
 		(width 0.2)
 		(layer "F.Cu")
@@
 	)
 	(segment
-		(start 131.75 106.55)
-		(end 131.75 108)
-		(width 0.2)
-		(layer "F.Cu")
-		(net "CAN_rocket_H")
-	)
-	(segment
 		(start 124.66 100.5)
 		(end 125.7 100.5)
@@
 		(net "CAN_rocket_H")
 	)
+	(segment
+		(start 131.5 106.3)
+		(end 131.5 108)
+		(width 0.2)
+		(layer "F.Cu")
+		(net "CAN_rocket_H")
+	)
 	(arc
 		(start 127.977132 103.765354)
@@
 	)
 	(segment
-		(start 121.66 100.5)
-		(end 128 106.84)
+		(start 128 110.25)
+		(end 129.75 112)
 		(width 0.5)
 		(layer "F.Cu")
@@
 	)
 	(segment
-		(start 128 110.25)
-		(end 129.75 112)
+		(start 128 106.84)
+		(end 128 110.25)
 		(width 0.5)
 		(layer "F.Cu")
@@
 	)
 	(segment
-		(start 135.5 110.75)
-		(end 135.5 108)
+		(start 121.66 100.5)
+		(end 128 106.84)
 		(width 0.5)
 		(layer "F.Cu")
@@
 	)
 	(segment
-		(start 128 106.84)
-		(end 128 110.25)
+		(start 134.25 112)
+		(end 135.5 110.75)
 		(width 0.5)
 		(layer "F.Cu")
@@
 	)
 	(segment
-		(start 134.25 112)
-		(end 135.5 110.75)
+		(start 135.5 110.75)
+		(end 135.5 108)
 		(width 0.5)
 		(layer "F.Cu")
@@
 	)
 	(segment
-		(start 153.46 109.45)
-		(end 153.46 100.625)
+		(start 145.7 111.3)
+		(end 151.61 111.3)
 		(width 0.5)
 		(layer "F.Cu")
@@
 	)
 	(segment
-		(start 145.7 111.3)
-		(end 151.61 111.3)
+		(start 153.46 100.625)
+		(end 153.5 100.585)
 		(width 0.5)
 		(layer "F.Cu")
@@
 	)
 	(segment
-		(start 144.85 108)
-		(end 144.85 110.45)
+		(start 144.5 110.1)
+		(end 145.7 111.3)
 		(width 0.5)
 		(layer "F.Cu")
@@
 	)
 	(segment
-		(start 153.5 100.585)
-		(end 153.44 100.525)
+		(start 153.46 109.45)
+		(end 153.46 100.625)
 		(width 0.5)
 		(layer "F.Cu")
@@
 	)
 	(segment
-		(start 144.85 110.45)
-		(end 145.7 111.3)
+		(start 153.5 100.585)
+		(end 153.44 100.525)
 		(width 0.5)
 		(layer "F.Cu")
@@
 	)
 	(segment
-		(start 153.46 100.625)
-		(end 153.5 100.585)
+		(start 144.5 108)
+		(end 144.5 110.1)
 		(width 0.5)
 		(layer "F.Cu")
@@
 	)
 	(segment
-		(start 146.75 108)
-		(end 146.75 100.775)
+		(start 146.5 101.025)
+		(end 150 97.525)
 		(width 0.5)
 		(layer "F.Cu")
@@
 	)
 	(segment
-		(start 146.75 100.775)
-		(end 150 97.525)
+		(start 146.5 108)
+		(end 146.5 101.025)
 		(width 0.5)
 		(layer "F.Cu")
@@
 		(polygon
 			(pts
-				(xy 108.5 98.75) (xy 119.25 98.75) (xy 119.25 111.25) (xy 115.5 111.25) (xy 115.5 102.25) (xy 108.5 102.25)
+				(xy 108.5 98.75) (xy 119.5 98.75) (xy 119.5 111.25) (xy 115.5 111.25) (xy 115.5 102.25) (xy 108.5 102.25)
 			)
 		)
