File: gse_connector_board_outer/gse_connector_board_outer.kicad_pcb (KiCad board)
At the start: 2 copper layers, 59 x 27 mm, 11 parts, among them J1 arming_connector, J2 gse_com_connector, J3 chg_connector, J4 Conn_02x04_Top_Bottom, J5 Conn_02x02_Top_Bottom, J7 Conn_02x02_Top_Bottom, J8 Conn_02x02_Top_Bottom

Commit message: final touches
Parts:
- removed J4: Conn_02x04_Top_Bottom, Connector_Molex:Molex_Micro-Fit_3.0_43045-0800_2x04_P3.00mm_Horizontal
- removed JP1: SolderJumper_2_Bridged, Jumper:SolderJumper-2_P1.3mm_Bridged_RoundedPad1.0x1.5mm
- moved J8 8.25 mm to (133.8, 97.3)
- moved J7 5.75 mm to (118.8, 97.8)
- moved J5 4.90 mm to (148.6, 97.5)
- moved H2 4.00 mm to (156.0, 92.0)
- moved G*** 2.47 mm to (143.8, 90.5)
Connections:
- J2 pad 1: unconnected-(J2-Pin_1-Pad1) -> +V_EXT
- J8 pad 1: GND_EXT -> GND_rocket
- J8 pad 3: GSE_CANH -> CAN_rocket_L
- J8 pad 4: GSE_CANL -> CAN_rocket_H
Routing:
- net GSE_CANL: track 20.1 -> 0.00 mm, vias 1 -> 0
- net GSE_CANH: track 15.6 -> 0.00 mm
- net GSE_CAN_TERM: track 14.0 -> 0.00 mm, vias 1 -> 0
- net GND_rocket: track 23.9 -> 11.4 mm
- net GND_Arm: track 0.00 -> 11.5 mm
- net Voltage_Arm: track 21.1 -> 13.5 mm
- net CAN_rocket_L: track 13.0 -> 7.99 mm
- net disarm: track 13.5 -> 8.49 mm
- net CAN_rocket_H: track 13.1 -> 9.34 mm
- net +V_EXT: track 7.85 -> 11.3 mm
- added copper zone on B.Cu, net (none)
- removed copper zone on B.Cu, net GND_EXT
Other:
- board size 59 x 27 mm -> 55 x 27 mm
- board text added: "Darm"
- board text added: "rev2.1"
- board text removed: "Disarm"
- board text removed: "GC_H"
- board text removed: "GC_L"
- board text removed: "GC_TM"
- board text removed: "G_ex"
- board text removed: "G_roc"
- board text removed: "RC_H"
- board text removed: "RC_L"
- board text removed: "Vext"
- board text removed: "rev2"

Commit message: final ordered version
Parts:
- J1, J2, J3: footprint custom_parts:4_pin_mag_con_mv_adapt -> custom_parts:4_pin_mag_con_flat_mv_adapt
- moved J7 0.43 mm to (118.8, 97.3)
- moved G*** 0.23 mm to (143.8, 90.3)
- moved J5 0.18 mm to (148.6, 97.3)
Routing:
- net CAN_rocket_H: track 9.34 -> 9.92 mm
- added copper zone on B.Cu, net GND_rocket
- removed copper zone on B.Cu, net (none)
