File: gse_connector_board_outer/gse_connector_board_outer.kicad_sch (KiCad schematic)
At the start: 11 parts, among them J1 arming_connector, J2 gse_com_connector, J3 chg_connector, J4 Conn_02x04_Top_Bottom, J5 Conn_02x02_Top_Bottom, J7 Conn_02x02_Top_Bottom, J8 Conn_02x02_Top_Bottom, U1 ICS_CAN_Isolator

Commit message: final order version
Parts:
- J1, J2, J3: footprint custom_parts:4_pin_mag_con_mv_adapt -> custom_parts:4_pin_mag_con_flat_mv_adapt
Changed lines of the file:
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@@
 			)
 		)
-		(property "Footprint" "custom_parts:4_pin_mag_con_mv_adapt"
+		(property "Footprint" "custom_parts:4_pin_mag_con_flat_mv_adapt"
 			(at 181.61 82.55 0)
 			(hide yes)
@@
 			)
 		)
-		(property "Footprint" "custom_parts:4_pin_mag_con_mv_adapt"
+		(property "Footprint" "custom_parts:4_pin_mag_con_flat_mv_adapt"
 			(at 154.94 82.55 0)
 			(hide yes)
@@
 			)
 		)
-		(property "Footprint" "custom_parts:4_pin_mag_con_mv_adapt"
+		(property "Footprint" "custom_parts:4_pin_mag_con_flat_mv_adapt"
 			(at 123.19 82.55 0)
 			(hide yes)
